File: ILJJ_Mk-XVI.sch (KiCad schematic (older format))
At the start: 36 parts, among them J1 AudioJack3_Ground, J2 AudioJack3_Ground, J3 Barrel_Jack_Switch, J4 AudioJack3_Ground, U1 NJM2114, U2 NJM2114

Commit message: [change] footprint size
Parts:
- C1: footprint Capacitors_ThroughHole:CP_Radial_D6.3mm_P2.50mm -> Capacitors_ThroughHole:CP_Radial_D8.0mm_P3.50mm
- C7: footprint Capacitors_ThroughHole:CP_Radial_D5.0mm_P2.00mm -> Capacitors_ThroughHole:CP_Radial_D6.3mm_P2.50mm
Changed lines of the file:
@@
 F 0 "C1" H 2488 5946 50  0000 L CNN
 F 1 "CP" H 2450 5800 50  0000 L CNN
-F 2 "Capacitors_ThroughHole:CP_Radial_D6.3mm_P2.50mm" H 2400 5900 50  0001 C CNN
+F 2 "Capacitors_ThroughHole:CP_Radial_D8.0mm_P3.50mm" H 2400 5900 50  0001 C CNN
 F 3 "~" H 2400 5900 50  0001 C CNN
 	1    2400 5900
@@
 F 0 "C7" H 5038 6096 50  0000 L CNN
 F 1 "CP" H 5050 6000 50  0000 L CNN
-F 2 "Capacitors_ThroughHole:CP_Radial_D5.0mm_P2.00mm" H 4950 6050 50  0001 C CNN
+F 2 "Capacitors_ThroughHole:CP_Radial_D6.3mm_P2.50mm" H 4950 6050 50  0001 C CNN
 F 3 "~" H 4950 6050 50  0001 C CNN
 	1    4950 6050

Commit message: [add] footprint for resistors and OPamps
Parts:
- R1, R10, R11, R12, R13, R14, R15, R16, R17, R2, R3, R4, R5, R6, R7, R8, R9: footprint (none) -> Resistors_ThroughHole:R_Axial_DIN0207_L6.3mm_D2.5mm_P2.54mm_Vertical
- U1, U2: footprint (none) -> Housings_DIP:DIP-8_W7.62mm_Socket
Changed lines of the file:
@@
 F 0 "U1" H 5650 1933 50  0000 C CNN
 F 1 "NJM2114" H 5650 2024 50  0000 C CNN
-F 2 "" H 5650 2300 50  0001 C CNN
+F 2 "Housings_DIP:DIP-8_W7.62mm_Socket" H 5650 2300 50  0001 C CNN
 F 3 "http://www.njr.com/semicon/PDF/NJM2114_E.pdf" H 5650 2300 50  0001 C CNN
 	1    5650 2300
@@
 F 0 "U2" H 6850 1933 50  0000 C CNN
 F 1 "NJM2114" H 6850 2024 50  0000 C CNN
-F 2 "" H 6850 2300 50  0001 C CNN
+F 2 "Housings_DIP:DIP-8_W7.62mm_Socket" H 6850 2300 50  0001 C CNN
 F 3 "http://www.njr.com/semicon/PDF/NJM2114_E.pdf" H 6850 2300 50  0001 C CNN
 	1    6850 2300
@@
 F 0 "U2" H 6850 3283 50  0000 C CNN
 F 1 "NJM2114" H 6850 3374 50  0000 C CNN
-F 2 "" H 6850 3650 50  0001 C CNN
+F 2 "Housings_DIP:DIP-8_W7.62mm_Socket" H 6850 3650 50  0001 C CNN
 F 3 "http://www.njr.com/semicon/PDF/NJM2114_E.pdf" H 6850 3650 50  0001 C CNN
 	2    6850 3650
@@
 F 0 "U1" H 5650 3283 50  0000 C CNN
 F 1 "NJM2114" H 5650 3374 50  0000 C CNN
-F 2 "" H 5650 3650 50  0001 C CNN
+F 2 "Housings_DIP:DIP-8_W7.62mm_Socket" H 5650 3650 50  0001 C CNN
 F 3 "http://www.njr.com/semicon/PDF/NJM2114_E.pdf" H 5650 3650 50  0001 C CNN
 	2    5650 3650
@@
 F 0 "R8" V 5443 1800 50  0000 C CNN
 F 1 "R" V 5534 1800 50  0000 C CNN
-F 2 "" V 5580 1800 50  0001 C CNN
+F 2 "Resistors_ThroughHole:R_Axial_DIN0207_L6.3mm_D2.5mm_P2.54mm_Vertical" V 5580 1800 50  0001 C CNN
 F 3 "~" H 5650 1800 50  0001 C CNN
 	1    5650 1800
@@
 F 0 "R12" V 6643 1800 50  0000 C CNN
 F 1 "R" V 6734 1800 50  0000 C CNN
-F 2 "" V 6780 1800 50  0001 C CNN
+F 2 "Resistors_ThroughHole:R_Axial_DIN0207_L6.3mm_D2.5mm_P2.54mm_Vertical" V 6780 1800 50  0001 C CNN
 F 3 "~" H 6850 1800 50  0001 C CNN
 	1    6850 1800
@@
 F 0 "R13" V 6643 3150 50  0000 C CNN
 F 1 "R" V 6734 3150 50  0000 C CNN
-F 2 "" V 6780 3150 50  0001 C CNN
+F 2 "Resistors_ThroughHole:R_Axial_DIN0207_L6.3mm_D2.5mm_P2.54mm_Vertical" V 6780 3150 50  0001 C CNN
 F 3 "~" H 6850 3150 50  0001 C CNN
 	1    6850 3150
@@
 F 0 "R9" V 5443 3150 50  0000 C CNN
 F 1 "R" V 5534 3150 50  0000 C CNN
-F 2 "" V 5580 3150 50  0001 C CNN
+F 2 "Resistors_ThroughHole:R_Axial_DIN0207_L6.3mm_D2.5mm_P2.54mm_Vertical" V 5580 3150 50  0001 C CNN
 F 3 "~" H 5650 3150 50  0001 C CNN
 	1    5650 3150
@@
 F 0 "R10" V 6043 2200 50  0000 C CNN
 F 1 "R" V 6134 2200 50  0000 C CNN
-F 2 "" V 6180 2200 50  0001 C CNN
+F 2 "Resistors_ThroughHole:R_Axial_DIN0207_L6.3mm_D2.5mm_P2.54mm_Vertical" V 6180 2200 50  0001 C CNN
 F 3 "~" H 6250 2200 50  0001 C CNN
 	1    6250 2200
@@
 F 0 "R11" V 6043 3550 50  0000 C CNN
 F 1 "R" V 6134 3550 50  0000 C CNN
-F 2 "" V 6180 3550 50  0001 C CNN
+F 2 "Resistors_ThroughHole:R_Axial_DIN0207_L6.3mm_D2.5mm_P2.54mm_Vertical" V 6180 3550 50  0001 C CNN
 F 3 "~" H 6250 3550 50  0001 C CNN
 	1    6250 3550
@@
 F 0 "U1" H 3608 5946 50  0000 L CNN
 F 1 "NJM2114" H 3608 5855 50  0000 L CNN
-F 2 "" H 3650 5900 50  0001 C CNN
+F 2 "Housings_DIP:DIP-8_W7.62mm_Socket" H 3650 5900 50  0001 C CNN
 F 3 "http://www.njr.com/semicon/PDF/NJM2114_E.pdf" H 3650 5900 50  0001 C CNN
 	3    3650 5900
@@
 F 0 "U2" H 4108 5946 50  0000 L CNN
 F 1 "NJM2114" H 4108 5855 50  0000 L CNN
-F 2 "" H 4150 5900 50  0001 C CNN
+F 2 "Housings_DIP:DIP-8_W7.62mm_Socket" H 4150 5900 50  0001 C CNN
 F 3 "http://www.njr.com/semicon/PDF/NJM2114_E.pdf" H 4150 5900 50  0001 C CNN
 	3    4150 5900
@@
 F 0 "R1" H 3159 5796 50  0000 L CNN
 F 1 "R_LED" H 3159 5705 50  0000 L CNN
-F 2 "" H 3100 5750 50  0001 C CNN
+F 2 "Resistors_ThroughHole:R_Axial_DIN0207_L6.3mm_D2.5mm_P2.54mm_Vertical" H 3100 5750 50  0001 C CNN
 F 3 "~" H 3100 5750 50  0001 C CNN
 	1    3100 5750
@@
 F 0 "R6" H 4609 5796 50  0000 L CNN
 F 1 "R" H 4609 5705 50  0000 L CNN
-F 2 "" H 4550 5750 50  0001 C CNN
+F 2 "Resistors_ThroughHole:R_Axial_DIN0207_L6.3mm_D2.5mm_P2.54mm_Vertical" H 4550 5750 50  0001 C CNN
 F 3 "~" H 4550 5750 50  0001 C CNN
 	1    4550 5750
@@
 F 0 "R7" H 4609 6096 50  0000 L CNN
 F 1 "R" H 4609 6005 50  0000 L CNN
-F 2 "" H 4550 6050 50  0001 C CNN
+F 2 "Resistors_ThroughHole:R_Axial_DIN0207_L6.3mm_D2.5mm_P2.54mm_Vertical" H 4550 6050 50  0001 C CNN
 F 3 "~" H 4550 6050 50  0001 C CNN
 	1    4550 6050
@@
 F 0 "R2" V 4293 1800 50  0000 C CNN
 F 1 "R" V 4384 1800 50  0000 C CNN
-F 2 "" V 4430 1800 50  0001 C CNN
+F 2 "Resistors_ThroughHole:R_Axial_DIN0207_L6.3mm_D2.5mm_P2.54mm_Vertical" V 4430 1800 50  0001 C CNN
 F 3 "~" H 4500 1800 50  0001 C CNN
 	1    4500 1800
@@
 F 0 "R3" V 4293 2300 50  0000 C CNN
 F 1 "R" V 4384 2300 50  0000 C CNN
-F 2 "" V 4430 2300 50  0001 C CNN
+F 2 "Resistors_ThroughHole:R_Axial_DIN0207_L6.3mm_D2.5mm_P2.54mm_Vertical" V 4430 2300 50  0001 C CNN
 F 3 "~" H 4500 2300 50  0001 C CNN
 	1    4500 2300
@@
 F 0 "R4" V 4293 3150 50  0000 C CNN
 F 1 "R" V 4384 3150 50  0000 C CNN
-F 2 "" V 4430 3150 50  0001 C CNN
+F 2 "Resistors_ThroughHole:R_Axial_DIN0207_L6.3mm_D2.5mm_P2.54mm_Vertical" V 4430 3150 50  0001 C CNN
 F 3 "~" H 4500 3150 50  0001 C CNN
 	1    4500 3150
@@
 F 0 "R5" V 4293 3650 50  0000 C CNN
 F 1 "R" V 4384 3650 50  0000 C CNN
-F 2 "" V 4430 3650 50  0001 C CNN
+F 2 "Resistors_ThroughHole:R_Axial_DIN0207_L6.3mm_D2.5mm_P2.54mm_Vertical" V 4430 3650 50  0001 C CNN
 F 3 "~" H 4500 3650 50  0001 C CNN
 	1    4500 3650
@@
 F 0 "R14" V 7993 2400 50  0000 C CNN
 F 1 "R" V 8084 2400 50  0000 C CNN
-F 2 "" V 8130 2400 50  0001 C CNN
+F 2 "Resistors_ThroughHole:R_Axial_DIN0207_L6.3mm_D2.5mm_P2.54mm_Vertical" V 8130 2400 50  0001 C CNN
 F 3 "~" H 8200 2400 50  0001 C CNN
 	1    8200 2400
@@
 F 0 "R16" V 8543 2550 50  0000 C CNN
 F 1 "R" V 8634 2550 50  0000 C CNN
-F 2 "" V 8680 2550 50  0001 C CNN
+F 2 "Resistors_ThroughHole:R_Axial_DIN0207_L6.3mm_D2.5mm_P2.54mm_Vertical" V 8680 2550 50  0001 C CNN
 F 3 "~" H 8750 2550 50  0001 C CNN
 	1    8750 2550
@@
 F 0 "R15" V 7993 3050 50  0000 C CNN
 F 1 "R" V 8084 3050 50  0000 C CNN
-F 2 "" V 8130 3050 50  0001 C CNN
+F 2 "Resistors_ThroughHole:R_Axial_DIN0207_L6.3mm_D2.5mm_P2.54mm_Vertical" V 8130 3050 50  0001 C CNN
 F 3 "~" H 8200 3050 50  0001 C CNN
 	1    8200 3050
@@
 F 0 "R17" V 8543 3200 50  0000 C CNN
 F 1 "R" V 8634 3200 50  0000 C CNN
-F 2 "" V 8680 3200 50  0001 C CNN
+F 2 "Resistors_ThroughHole:R_Axial_DIN0207_L6.3mm_D2.5mm_P2.54mm_Vertical" V 8680 3200 50  0001 C CNN
 F 3 "~" H 8750 3200 50  0001 C CNN
 	1    8750 3200
