File: ILJJ_Mk-XVI.sch (KiCad schematic (older format))
At the start: 36 parts, among them J1 AudioJack3_Ground, J2 AudioJack3_Ground, J3 Barrel_Jack_Switch, J4 AudioJack3_Ground, U1 NJM2114, U2 NJM2114

Commit message: [add] assigned footprints for connectors
Parts:
- J1, J2, J4: footprint (none) -> footprints:MJ-8435
- J3: footprint (none) -> Connect:BARREL_JACK
Changed lines of the file:
@@
 F 0 "J1" H 1800 1700 50  0000 C CNN
 F 1 "AudioJack3_Ground" H 1800 1800 50  0000 C CNN
-F 2 "" H 1800 2100 50  0001 C CNN
+F 2 "footprints:MJ-8435" H 1800 2100 50  0001 C CNN
 F 3 "~" H 1800 2100 50  0001 C CNN
 	1    1800 2100
@@
 F 0 "J4" H 9550 2350 50  0000 R CNN
 F 1 "AudioJack3_Ground" H 9850 2450 50  0000 R CNN
-F 2 "" H 9500 2750 50  0001 C CNN
+F 2 "footprints:MJ-8435" H 9500 2750 50  0001 C CNN
 F 3 "~" H 9500 2750 50  0001 C CNN
 	1    9500 2750
@@
 F 0 "J3" H 1950 5400 50  0000 C CNN
 F 1 "Barrel_Jack_Switch" H 1950 5500 50  0000 C CNN
-F 2 "" H 2000 5660 50  0001 C CNN
+F 2 "Connect:BARREL_JACK" H 2000 5660 50  0001 C CNN
 F 3 "~" H 2000 5660 50  0001 C CNN
 	1    1950 5700
@@
 F 0 "J2" H 1800 3050 50  0000 C CNN
 F 1 "AudioJack3_Ground" H 1800 3150 50  0000 C CNN
-F 2 "" H 1800 3450 50  0001 C CNN
+F 2 "footprints:MJ-8435" H 1800 3450 50  0001 C CNN
 F 3 "~" H 1800 3450 50  0001 C CNN
 	1    1800 3450

Commit message: [add] footprints for RV
Parts:
- RV1, RV2, RV3: footprint (none) -> footprints:RS30112AJA02
Changed lines of the file:
@@
 F 0 "RV1" V 2700 1850 50  0000 R CNN
 F 1 "R_POT_Dual" V 2800 1850 50  0000 R CNN
-F 2 "" H 3150 1975 50  0001 C CNN
+F 2 "footprints:RS30112AJA02" H 3150 1975 50  0001 C CNN
 F 3 "~" H 3150 1975 50  0001 C CNN
 	1    2900 2050
@@
 F 0 "RV3" V 7804 2612 50  0000 R CNN
 F 1 "R_POT_Dual" V 7895 2612 50  0000 R CNN
-F 2 "" H 8100 2725 50  0001 C CNN
+F 2 "footprints:RS30112AJA02" H 8100 2725 50  0001 C CNN
 F 3 "~" H 8100 2725 50  0001 C CNN
 	1    7850 2800
@@
 F 0 "RV2" V 2700 3200 50  0000 R CNN
 F 1 "R_POT_Dual" V 2800 3200 50  0000 R CNN
-F 2 "" H 3150 3325 50  0001 C CNN
+F 2 "footprints:RS30112AJA02" H 3150 3325 50  0001 C CNN
 F 3 "~" H 3150 3325 50  0001 C CNN
 	1    2900 3400

Commit message: [remove] 増幅回路を一段削減
反転しててもええやろ(適当)
Parts:
- removed R10, R11, R12, R13: R, Resistors_ThroughHole:R_Axial_DIN0207_L6.3mm_D2.5mm_P2.54mm_Vertical, symbol Device:R
- removed U2: NJM2114, Housings_DIP:DIP-8_W7.62mm_Socket, symbol Amplifier_Operational:NJM2114
Connections:
- wire segments 94 -> 76

Commit message: [change] some footprints
Parts:
- C2: footprint Capacitors_SMD:C_0603_HandSoldering -> Capacitors_ThroughHole:C_Disc_D9.0mm_W5.0mm_P5.00mm
Changed lines of the file:
@@
 $EndComp
-Wire Wire Line
-	6750 2700 6750 2550
-Wire Wire Line
-	6550 2700 6750 2700
 Wire Wire Line
 	6550 3200 6750 3200
@@
 F 0 "C2" H 2842 5946 50  0000 L CNN
 F 1 "C" H 2800 5800 50  0000 L CNN
-F 2 "Capacitors_SMD:C_0603_HandSoldering" H 2750 5900 50  0001 C CNN
+F 2 "Capacitors_ThroughHole:C_Disc_D9.0mm_W5.0mm_P5.00mm" H 2750 5900 50  0001 C CNN
 F 3 "~" H 2750 5900 50  0001 C CNN
 	1    2750 5900
@@
 F 3 "~" H 4000 6050 50  0001 C CNN
 	1    4000 6050
-	1    0    0    -1
+	1    0    0    1
 $EndComp
 Wire Wire Line
@@
 Wire Wire Line
 	4650 3550 4650 3650
-Connection ~ 6750 2550
 $Comp
 L Device:C C8
@@
 	6850 2400 6750 2400
 Wire Wire Line
-	6750 2400 6750 2550
-Wire Wire Line
 	7450 2400 7550 2400
 $Comp
@@
 	7900 2650 8100 2650
 Connection ~ 7550 2400
-Connection ~ 6750 3050
 NoConn ~ 2250 5700
 Wire Wire Line
@@
 Wire Wire Line
 	5950 2300 5950 2700
-Wire Wire Line
-	5950 2700 6550 2700
-Connection ~ 6550 2700
 Wire Wire Line
 	6550 1800 6550 2400
@@
 Connection ~ 5350 3550
 Connection ~ 4650 3550
+Connection ~ 6550 2700
+Connection ~ 6750 3050
+Connection ~ 6750 2550
+Wire Wire Line
+	5950 2700 6550 2700
+Wire Wire Line
+	6550 2700 6750 2700
+Wire Wire Line
+	6750 2400 6750 2550
+Wire Wire Line
+	6750 2700 6750 2550
 $EndSCHEMATC
