File: ILJJ_Mk-XVI.kicad_pcb (KiCad board)
At the start: 2 copper layers, 60.5 x 50 mm, 31 parts, among them J1 AudioJack3_Ground, J2 AudioJack3_Ground, J3 Barrel_Jack_Switch, J4 AudioJack3_Ground, U1 NJM2114

Commit message: [add] 配線
Parts:
- moved C1 0.25 mm to (195.5, 119.5)
Routing:
- net GND: track 0.00 -> 147.8 mm, vias 0 -> 1
- net Net-(R15-Pad1): track 0.00 -> 80.2 mm, vias 0 -> 1
- net Net-(R14-Pad1): track 0.00 -> 78.0 mm, vias 0 -> 2
- net VCC: track 0.00 -> 41.6 mm
- net 4.5V: track 0.00 -> 41.3 mm
- net Net-(R4-Pad1): track 0.00 -> 38.9 mm
- net CH2_R: track 0.00 -> 38.4 mm, vias 0 -> 1
- net Net-(R2-Pad1): track 0.00 -> 35.0 mm
- net CH2_L: track 0.00 -> 30.9 mm, vias 0 -> 1
- net CH1_R: track 0.00 -> 28.9 mm
- net Net-(R9-Pad1): track 0.00 -> 25.8 mm, vias 0 -> 2
- net Net-(R8-Pad1): track 0.00 -> 24.5 mm, vias 0 -> 1
- net Net-(J2-PadR): track 0.00 -> 19.4 mm
- net Net-(J1-PadR): track 0.00 -> 19.4 mm
- net Net-(D1-Pad2): track 0.00 -> 19.0 mm, vias 0 -> 1
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